File: H_bridge_PCB_Design/H_bridge_PCB.kicad_pcb (KiCad board)
At the start: 2 copper layers, 100 x 100 mm, 105 parts, among them IC2 L7812ABD2T-TR, IC5 ACS37800KMACTR-030B3-I2C, J1 TMS-102-21-G-S, J2 TMS-102-21-G-S, J3 TMS-102-21-G-S, J4 TMS-102-21-G-S, J5 TMS-102-21-G-S, P1 USB_C_Plug_USB2.0, Q1 IRLB4030PBF, Q10 IPD90N10S4L06ATMA1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

Commit message: Updated PCB design files
Parts:
- added C16: MKS4C042204C00KSSD, SamacSys_Parts:MKS4C042204C00KSSD, F.Cu at (115.2, 102.2)
- added C22: MKS4C042204C00KSSD, SamacSys_Parts:MKS4C042204C00KSSD, F.Cu at (115.2, 118.2)
- added J10: TMS-102-21-G-S, SamacSys_Parts:TMS-102-YY-XX-S, F.Cu at (106.2, 103.8)
- added J11: TMS-102-21-G-S, SamacSys_Parts:TMS-102-YY-XX-S, F.Cu at (135.2, 100.2)
- added J6: TMS-102-21-G-S, SamacSys_Parts:TMS-102-YY-XX-S, F.Cu at (135.2, 106.2)
- added J7: TMS-102-21-G-S, SamacSys_Parts:TMS-102-YY-XX-S, F.Cu at (106.2, 108.8)
- added J8: TMS-102-21-G-S, SamacSys_Parts:TMS-102-YY-XX-S, F.Cu at (135.2, 113.7)
- added J9: TMS-102-21-G-S, SamacSys_Parts:TMS-102-YY-XX-S, F.Cu at (109.8, 115.0)
- C13: value MKP1847H55025JK2 -> MKS4C042204C00KSSD; footprint SamacSys_Parts:MKP1847H55025JK2 -> SamacSys_Parts:MKS4C042204C00KSSD
- moved C13 9.41 mm to (115.2, 110.2)
- moved L1 4.76 mm to (138.2, 65.3)
Connections:
- C13 pad 1: Out- -> Net-(C13-Pad1)
- C13 pad 2: SV2 -> Net-(C13-Pad2)
- C4 pad 2: Out- -> Cout-
- C5 pad 2: Out- -> Cout-
- D3 pad 1: Out- -> Cout-
- D3 pad 2: Out- -> Cout-
- D5 pad 3: Out- -> Cout-
- IC5 pad 5: Out- -> Cout-
- IC5 pad 6: Out- -> Cout-
- IC5 pad 7: Out- -> Cout-
- IC5 pad 8: Out- -> Cout-
- L1 pad 2: SV2 -> Cout+
- Q10 pad 4: Out- -> Cout-
- Q3 pad 3: Out- -> Cout-
- Q4 pad 2: Out- -> Cout-
- Q9 pad 3: Out- -> Cout-
- R15 pad 2: SV2 -> Cout+
- R7 pad 2: Out- -> Cout-
- TP3 pad 1: SV2 -> Cout+
- U3 pad 6: Out- -> Cout-
Routing:
- net Cout-: track 0.00 -> 137.7 mm, vias 0 -> 4
- net Out-: track 131.8 -> 0.00 mm, vias 2 -> 0
- net SV2: track 82.7 -> 0.00 mm, vias 1 -> 0
- net Cout+: track 0.00 -> 65.7 mm, vias 0 -> 1
- net Net-(C16-Pad1): track 0.00 -> 13.4 mm
- net Net-(C13-Pad1): track 0.00 -> 12.8 mm
- net Net-(C13-Pad2): track 0.00 -> 12.6 mm
- net Net-(C16-Pad2): track 0.00 -> 11.0 mm
- net Net-(C22-Pad1): track 0.00 -> 6.85 mm
- net Net-(C22-Pad2): track 0.00 -> 6.35 mm
- net Out+: track 137.5 -> 142.3 mm
- added copper zone on F.Cu, net Cout-
- removed copper zone on F.Cu, net Out-
Other:
- board text added: "0-6.6µF"
- board text added: "2.2"
- board text added: "4.4"
- board text added: "6.6"

Commit message: Added picutres for bipolar and unipolar, changed pins for I2C-2
Connections:
- U1 pad 28: unconnected-(U1-IO17-Pad28) -> SDA2MC
- U1 pad 30: unconnected-(U1-IO18-Pad30) -> SCL2MC
- U1 pad 6: SDA2MC -> unconnected-(U1-IO34-Pad6)
- U1 pad 7: SCL2MC -> unconnected-(U1-IO35-Pad7)
Routing:
- net SDA2MC: track 9.10 -> 29.1 mm, vias 0 -> 2
- net SCL2MC: track 9.83 -> 24.6 mm, vias 0 -> 2
- net VUSB(5V): track 9.63 -> 15.8 mm, vias 2 -> 3
Changed lines of the file:
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@@
 	(net 57 "unconnected-(U1-IO5-Pad29)")
 	(net 58 "unconnected-(U1-SCK{slash}CLK-Pad20)")
-	(net 59 "unconnected-(U1-IO17-Pad28)")
+	(net 59 "unconnected-(U1-IO34-Pad6)")
 	(net 60 "unconnected-(U1-NC-Pad32)")
 	(net 61 "unconnected-(U1-IO23-Pad37)")
@@
 	(net 65 "HIN2")
 	(net 66 "unconnected-(U1-SCS{slash}CMD-Pad19)")
-	(net 67 "unconnected-(U1-IO18-Pad30)")
+	(net 67 "unconnected-(U1-IO35-Pad7)")
 	(net 68 "unconnected-(U1-IO2-Pad24)")
 	(net 69 "LIN1")
@@
 			(size 1.5 0.9)
 			(layers "F.Cu" "F.Paste" "F.Mask")
-			(net 50 "SDA2MC")
+			(net 59 "unconnected-(U1-IO34-Pad6)")
 			(pinfunction "IO34")
 			(pintype "input")
@@
 			(size 1.5 0.9)
 			(layers "F.Cu" "F.Paste" "F.Mask")
-			(net 49 "SCL2MC")
+			(net 67 "unconnected-(U1-IO35-Pad7)")
 			(pinfunction "IO35")
 			(pintype "input")
@@
 			(size 1.5 0.9)
 			(layers "F.Cu" "F.Paste" "F.Mask")
-			(net 59 "unconnected-(U1-IO17-Pad28)")
+			(net 50 "SDA2MC")
 			(pinfunction "IO17")
 			(pintype "bidirectional")
@@
 			(size 1.5 0.9)
 			(layers "F.Cu" "F.Paste" "F.Mask")
-			(net 67 "unconnected-(U1-IO18-Pad30)")
+			(net 49 "SCL2MC")
 			(pinfunction "IO18")
 			(pintype "bidirectional")
@@
 	)
 	(segment
+		(start 102.65 142.4)
+		(end 102.25 142)
+		(width 0.2)
+		(layer "F.Cu")
+		(net 12)
+	)
+	(segment
+		(start 102.65 143.255)
+		(end 102.65 142.4)
+		(width 0.2)
+		(layer "F.Cu")
+		(net 12)
+	)
+	(segment
 		(start 97.5 142)
 		(end 97.85 142.35)
@@
 	)
 	(via
+		(at 102.25 142)
+		(size 0.6)
+		(drill 0.3)
+		(layers "F.Cu" "B.Cu")
+		(net 12)
+	)
+	(via
 		(at 97.5 142)
 		(size 0.6)
@@
 	)
 	(segment
+		(start 102.25 142)
+		(end 97.5 142)
+		(width 0.2)
+		(layer "B.Cu")
+		(net 12)
+	)
+	(segment
 		(start 95 142)
 		(end 97.5 142)
@@
 	)
 	(segment
-		(start 80 140.215)
-		(end 80 136)
+		(start 81 135)
+		(end 83 133)
 		(width 0.2)
 		(layer "F.Cu")
@@
 	)
 	(segment
-		(start 78.75 140.515)
-		(end 79.7 140.515)
+		(start 66.5 136)
+		(end 64.57 137.93)
 		(width 0.2)
 		(layer "F.Cu")
@@
 	)
 	(segment
-		(start 80 136)
-		(end 83 133)
+		(start 64.57 137.93)
+		(end 61.3075 137.93)
 		(width 0.2)
 		(layer "F.Cu")
@@
 	)
 	(segment
-		(start 79.7 140.515)
-		(end 80 140.215)
+		(start 74 136)
+		(end 66.5 136)
 		(width 0.2)
 		(layer "F.Cu")
 		(net 49)
 	)
+	(via
+		(at 74 136)
+		(size 0.6)
+		(drill 0.3)
+		(layers "F.Cu" "B.Cu")
+		(net 49)
+	)
+	(via
+		(at 81 135)
+		(size 0.6)
+		(drill 0.3)
+		(layers "F.Cu" "B.Cu")
+		(net 49)
+	)
+	(segment
+		(start 75 137)
+		(end 74 136)
+		(width 0.2)
+		(layer "B.Cu")
+		(net 49)
+	)
+	(segment
+		(start 81 135)
+		(end 79 137)
+		(width 0.2)
+		(layer "B.Cu")
+		(net 49)
+	)
+	(segment
+		(start 76.25 137)
+		(end 75 137)
+		(width 0.2)
+		(layer "B.Cu")
+		(net 49)
+	)
+	(segment
+		(start 79 137)
+		(end 76.25 137)
+		(width 0.2)
+		(layer "B.Cu")
+		(net 49)
+	)
 	(segment
 		(start 81 137)
@@
 	)
 	(segment
-		(start 78.75 141.785)
-		(end 79.7 141.785)
+		(start 69.36 135.39)
+		(end 61.3075 135.39)
 		(width 0.2)
 		(layer "F.Cu")
@@
 	)
 	(segment
-		(start 79.7 141.785)
-		(end 81 140.485)
+		(start 81 141)
+		(end 80.75 141.25)
+		(width 0.2)
+		(layer "F.Cu")
+		(net 50)
+	)
+	(segment
+		(start 81 140.485)
+		(end 81 141)
 		(width 0.2)
 		(layer "F.Cu")
 		(net 50)
 	)
+	(via
+		(at 69.36 135.39)
+		(size 0.6)
+		(drill 0.3)
+		(layers "F.Cu" "B.Cu")
+		(net 50)
+	)
+	(via
+		(at 80.75 141.25)
+		(size 0.6)
+		(drill 0.3)
+		(layers "F.Cu" "B.Cu")
+		(net 50)
+	)
+	(segment
+		(start 69.89 135.39)
+		(end 75.75 141.25)
+		(width 0.2)
+		(layer "B.Cu")
+		(net 50)
+	)
+	(segment
+		(start 75.75 141.25)
+		(end 80.75 141.25)
+		(width 0.2)
+		(layer "B.Cu")
+		(net 50)
+	)
+	(segment
+		(start 69.36 135.39)
+		(end 69.89 135.39)
+		(width 0.2)
+		(layer "B.Cu")
+		(net 50)
+	)
 	(segment
 		(start 56 66)
@@
 	)
 	(segment
-		(start 68.165 134.165)
-		(end 61.25 134.165)
+		(start 75 134)
+		(end 68.33 134)
 		(width 0.2)
 		(layer "F.Cu")
@@
 	)
 	(segment
-		(start 90.905 127.65)
-		(end 90.905 129.845)
+		(start 68.165 134.165)
+		(end 61.25 134.165)
 		(width 0.2)
 		(layer "F.Cu")
@@
 	)
 	(segment
-		(start 75 134)
-		(end 68.33 134)
+		(start 90.905 127.65)
+		(end 90.905 129.845)
 		(width 0.2)
 		(layer "F.Cu")
