File: H_bridge_PCB_Design/H_bridge_PCB.kicad_pcb (KiCad board)
At the start: 2 copper layers, 110.2 x 110.2 mm, 128 parts, among them IC1 LM2671M-3.3_NOPB, IC2 L7812ABD2T-TR, IC5 ACS37800KMACTR-030B3-I2C, J1 TSW-102-15-T-S, J12 TSW-102-15-T-S, J13 1734510-1, J14 TSW-102-15-T-S, J15 TSW-102-15-T-S, J2 TSW-102-15-T-S, J3 TSW-102-15-T-S, J4 TSW-102-15-T-S, J5 TSW-102-15-T-S, J7 TSW-102-15-T-S, J9 TSW-102-15-T-S, Q1 IRLB4030PBF, Q10 IPD90N10S4L06ATMA1, Q11 NTR2101P, Q12 NTR2101P, Q2 IRLB4030PBF, Q3 IRLB4030PBF, Q4 IRLB4030PBF, Q5 IPD90N10S4L06ATMA1, Q6 IPD90N10S4L06ATMA1, Q7 BC817, Q8 BC817, Q9 IPD90N10S4L06ATMA1, U1 ESP32-WROOM-32, U2 IR2110S, U3 IR2110S, U4 INA228, U5 LTC4412xS6, U6 LD1086DT50TR, U7 CH340C, U8 3544-2, U9 LT1963AxST-3.3

Commit message: huge changes output measurement
Parts:
- removed D13: S210, SamacSys_Parts:DIOM5336X265N
- removed IC5: ACS37800KMACTR-030B3-I2C, SamacSys_Parts:ACS37002LMCA050U5
- removed L1: IFDC3030EZER101M, SamacSys_Parts:IFDC3030EZER101M
- removed Q11, Q12: NTR2101P, Package_TO_SOT_SMD:SOT-23
- removed R38, R39: 10k, Resistor_SMD:R_0805_2012Metric_Pad1.20x1.40mm_HandSolder
- removed R43, R44: 1M, Resistor_SMD:R_0805_2012Metric_Pad1.20x1.40mm_HandSolder
- removed R45: 20k, Resistor_SMD:R_0805_2012Metric_Pad1.20x1.40mm_HandSolder
- removed R46, R47, R48, R49: 0, Resistor_SMD:R_0805_2012Metric_Pad1.20x1.40mm_HandSolder
- removed U9: LT1963AxST-3.3, Package_TO_SOT_SMD:SOT-223-3_TabPin2
- added C33: 100 nF, Resistor_SMD:R_0805_2012Metric_Pad1.20x1.40mm_HandSolder, F.Cu at (152.2, 130.8)
- added C34: 1 µF, Resistor_SMD:R_0805_2012Metric_Pad1.20x1.40mm_HandSolder, F.Cu at (154.6, 130.8)
- added C35: 100 nF, Resistor_SMD:R_0805_2012Metric_Pad1.20x1.40mm_HandSolder, F.Cu at (143.8, 128.2)
- added C36: 1 µF, Resistor_SMD:R_0805_2012Metric_Pad1.20x1.40mm_HandSolder, F.Cu at (141.8, 128.2)
- added IC3: AMC1306M25DWVR, SamacSys_Parts:SOIC127P1150X280-8N, F.Cu at (140.9, 136.9)
- added LED4: TLMG1100-GS15-1, Resistor_SMD:R_0805_2012Metric_Pad1.20x1.40mm_HandSolder, F.Cu at (66.8, 112.0)
- added PS1: NXJ1S0303MC-R13, SamacSys_Parts:NXJ1S0303MCR13, F.Cu at (130.5, 139.4)
- added R17: 1k, Resistor_SMD:R_0805_2012Metric_Pad1.20x1.40mm_HandSolder, F.Cu at (146.6, 127.8)
- C11: value 10 nF -> 1µF
- C19: footprint Capacitor_SMD:C_0805_2012Metric -> Resistor_SMD:R_0805_2012Metric_Pad1.20x1.40mm_HandSolder
- C22: value 100uF -> 100 nF; footprint SamacSys_Parts:EEE1AA101SP -> Resistor_SMD:R_0805_2012Metric_Pad1.20x1.40mm_HandSolder
- C31, C32: value 1µF -> 1 µF
- IC1: value LM2671M-3.3_NOPB -> AMC1306M25DWVR; footprint SamacSys_Parts:SOIC127P600X175-8N -> SamacSys_Parts:SOIC127P1150X280-8N
- R11: value 470k -> 100
- R15: value 1M -> GMR100HTBFER015; footprint Resistor_SMD:R_0805_2012Metric_Pad1.20x1.40mm_HandSolder -> Resistor_SMD:R_2512_6332Metric_Pad1.40x3.35mm_HandSolder
- R16: value 1M -> 120k
- U5: value LTC4412xS6 -> LT1963AxST-3.3; footprint Package_TO_SOT_SMD:TSOT-23-6 -> Package_TO_SOT_SMD:SOT-223-3_TabPin2
- moved C22 95.5 mm to (144.2, 146.8)
- moved IC1 86.1 mm to (147.8, 136.9), turned to -90 degrees
- moved C31 62.2 mm to (153.2, 137.6)
- moved C32 52.6 mm to (144.2, 144.8)
- moved J4 52.4 mm to (60.4, 108.4), turned to 180 degrees
- moved C11 44.2 mm to (97.8, 147.0), turned to 90 degrees
- moved R11 40.2 mm to (66.8, 116.0), turned to 90 degrees
- moved J12 18.5 mm to (120.2, 130.0)
- moved C19 17.2 mm to (153.2, 139.6), turned to 180 degrees
- moved R15 15.2 mm to (134.2, 127.4)
- moved R16 13.3 mm to (150.4, 127.8), turned to 180 degrees
- moved LED1 7.16 mm to (68.8, 112.0)
- moved LED2 7.16 mm to (72.8, 112.0)
- moved LED3 7.16 mm to (70.8, 112.0)
- moved R27 7.16 mm to (68.8, 116.0)
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Connections:
- C11 pad 1: Net-(IC1-CB) -> +3.3V
- C11 pad 2: Net-(D13-K) -> GND
- C18 pad 1: VIN(3.3V) -> +3.3V
- C19 pad 1: +3.3V -> GND
- C19 pad 2: GND -> +3.3V
- C22 pad 1: SI1 -> GND
- C22 pad 2: GND -> +3.3V
- C23 pad 1: VIN(3.3V) -> +3.3V
- C27 pad 1: VIN(3.3V) -> +3.3V
- C31 pad 1: VUSB(3.3V) -> GND
- C31 pad 2: GND -> +3.3V
- C32 pad 1: +3.3V -> GND
- C32 pad 2: GND -> +3.3V
- IC1 pad 1: Net-(IC1-CB) -> 3.3_Sensor
- IC1 pad 2: unconnected-(IC1-SS-Pad2) -> Net-(IC1-AINP)
- IC1 pad 3: unconnected-(IC1-SYNC-Pad3) -> SI2
- IC1 pad 4: VIN(3.3V) -> SI2
- IC1 pad 5: unconnected-(IC1-ON/~{OFF}-Pad5) -> GND
- IC1 pad 6: GND -> Data_V
- IC1 pad 7: SI1 -> CLK_V
- IC1 pad 8: Net-(D13-K) -> +3.3V
- J12 pad 1: DIO_0 -> CLK_V
- J12 pad 2: DIO_1 -> Data_V
- J5 pad 1: SCL2 -> Data_C
- J5 pad 2: SDA2 -> CLK_C
- R11 pad 1: +3.3V -> GND
- R11 pad 2: Net-(Q12-G) -> Net-(LED4-K)
- R15 pad 1: Net-(R15-Pad1) -> Cout-
- R15 pad 2: Cout+ -> SI2
- R16 pad 1: Net-(R16-Pad1) -> Cout+
- R16 pad 2: SI2 -> Net-(IC1-AINP)
- U1 pad 10: DIO_0 -> CLK_C
- U1 pad 11: DIO_1 -> Data_C
- U1 pad 28: SDA2MC -> CLK_V
- U1 pad 30: SCL2MC -> Data_V
- U1 pad 31: unconnected-(U1-IO19-Pad31) -> SatusLED
- U4 pad 6: VIN(3.3V) -> +3.3V
- U5 pad 1: VUSB(3.3V) -> VUSB(5V)
- U5 pad 3: GND -> +3.3V
Routing:
- net VIN(3.3V): track 136.0 -> 0.00 mm, vias 6 -> 0
- net CLK_V: track 0.00 -> 102.4 mm, vias 0 -> 4
- net Data_V: track 0.00 -> 99.0 mm, vias 0 -> 5
- net CLK_C: track 0.00 -> 80.2 mm, vias 0 -> 6
- net +3.3V: track 180.8 -> 258.0 mm, vias 9 -> 6
- net Data_C: track 0.00 -> 75.8 mm, vias 0 -> 6
- net SCL2: track 67.3 -> 0.00 mm, vias 3 -> 0
- net SDA2: track 66.5 -> 0.00 mm
- net DIO_0: track 63.9 -> 0.00 mm, vias 6 -> 0
- net DIO_1: track 62.3 -> 0.00 mm, vias 6 -> 0
- net SCL1: track 132.5 -> 77.6 mm, vias 11 -> 5
- net SDA1: track 135.1 -> 81.0 mm, vias 8 -> 4
- net SatusLED: track 0.00 -> 44.1 mm, vias 0 -> 2
- net 3.3_Sensor: track 0.00 -> 43.6 mm
- net Net-(D13-K): track 29.5 -> 0.00 mm, vias 4 -> 0
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Other:
- board text added: "12V - LDO"
- board text added: "3.3V LDO"
- board text added: "CLK_C"
- board text added: "CLK_V"
- board text added: "DC Link Capacitors"
- board text added: "D_C"
- board text added: "D_V"
- board text added: "Filter - C"
- board text added: "Filter - L"
- board text added: "Gatedrivers"
- board text added: "Meas Input"
- board text added: "Meas Output"
- board text added: "Mosfet1"
- board text added: "Mosfet2"
- board text added: "Mosfet3"
- board text added: "Mosfet4"
- board text added: "Out+"
- board text added: "Out-"
- board text added: "Overvoltage protection"
- board text added: "Status"
- board text added: "USB connection"
- board text removed: "2.2"
- board text removed: "DIO_0"
- board text removed: "DIO_1"
- board text removed: "SC-L"
- board text removed: "SCL1"
- board text removed: "SDA2"

Commit message: new pcb
Parts:
- removed U8: 3544-2, SamacSys_Parts:3544-2
- added R18: 12k, Resistor_SMD:R_0805_2012Metric_Pad1.20x1.40mm_HandSolder, F.Cu at (70.2, 82.8)
- added R19: 0, Resistor_SMD:R_0805_2012Metric_Pad1.20x1.40mm_HandSolder, F.Cu at (65.6, 105.0)
- added R20: 0, Resistor_SMD:R_0805_2012Metric_Pad1.20x1.40mm_HandSolder, F.Cu at (67.8, 105.0)
- added S1: B3U-1000P, SamacSys:B3U-1000P, F.Cu at (77.0, 115.6)
- D1, D2, D3, D5: footprint SamacSys_Parts:FSV2060L -> SamacSys:FSV2060L
- IC1, IC3: footprint SamacSys_Parts:SOIC127P1150X280-8N -> SamacSys:SOIC127P1150X280-8N
- IC2: footprint SamacSys_Parts:L7812ABD2TTR -> SamacSys:L7812ABD2TTR
- PS1: footprint SamacSys_Parts:NXJ1S0303MCR13 -> SamacSys:NXJ1S0303MCR13
- Q1, Q2, Q3, Q4: footprint SamacSys_Parts:TO254P483X1016X1994-3P -> SamacSys:TO254P483X1016X1994-3P
- Q10, Q5, Q6, Q9: footprint SamacSys_Parts:IPD90N10S4L06ATMA1 -> SamacSys:IPD90N10S4L06ATMA1
Connections:
- TP1 pad 1: Net-(TP1-Pad1) -> SI1
- U1 pad 31: SatusLED -> StatusLED
- U1 pad 33: unconnected-(U1-IO21-Pad33) -> Shutoff1
- U2 pad 13: GND -> Shutoff
- U3 pad 13: GND -> Shutoff
- U4 pad 3: unconnected-(U4-~{Alert}-Pad3) -> Shutoff1
Routing:
- net Shutoff1: track 0.00 -> 81.2 mm, vias 0 -> 8
- net Shutoff: track 0.00 -> 44.8 mm, vias 0 -> 6
- net EN: track 17.6 -> 49.9 mm, vias 0 -> 2
- net Net-(TP1-Pad1): track 11.9 -> 0.00 mm
- net SI1: track 61.0 -> 71.2 mm
- net GND: track 245.4 -> 241.7 mm, vias 35 -> 37
- net +5V: track 83.2 -> 80.2 mm
- net +3.3V: track 258.0 -> 259.8 mm
- net HIN2: track 30.3 -> 29.5 mm
Other:
- board text added: "Reset"
