File: H_bridge_PCB_Design/voltage_source.kicad_sch (KiCad schematic)
At the start: 21 parts, among them IC2 L7812ABD2T-TR, U5 LD1086DT33TR, U6 LD1086DT50TR, U8 3544-2

Commit message: Interrupt for PWM and unipolar modulation
Parts:
- removed U5: LD1086DT33TR, Package_TO_SOT_SMD:TO-252-2, symbol Regulator_Linear:LD1086DT33TR
- added C22: 100uF, SamacSys_Parts:EEE1AA101SP, symbol Device:C_Polarized_Small_US
- added D12: HPZR-C26X, SamacSys_Parts:HPZRC26X, symbol SamacSys_Parts:HPZR-C26X
- added D13: S210, SamacSys_Parts:DIOM5336X265N, symbol SamacSys_Parts:S210
- added IC1: LM2671M-3.3_NOPB, SOIC127P600X175-8N, symbol SamacSys_Parts:LM2671M-3.3_NOPB
- added J15: TSW-102-15-T-S, SamacSys_Parts:TSW-102-XX-YY-S, symbol SamacSys_Parts:TSW-102-15-T-S
- added L1: IFDC3030EZER101M, SamacSys_Parts:IFDC3030EZER101M, symbol SamacSys_Parts:IFDC3030EZER101M
- added R12: 1, Resistor_SMD:R_0805_2012Metric_Pad1.20x1.40mm_HandSolder, symbol Device:R
- C11: value 1µF -> 10 nF
Connections:
- net +24V: now also C22.1, IC1.7 (VIN); no longer C11.1
- net +3.3V: now also IC1.4 (FB), J15.1, L1.2
- net GND: now also C22.2, D13.2 (A), IC1.6 (GND), J15.2, R12.2; no longer C11.2
- new net: D12.2 (A), R12.1
- new net: C11.1, IC1.1 (CB)
- new net: C11.2, D13.1 (K), IC1.8 (VSW), L1.1
- new net SO1: D12.1 (K)
Other:
- moved on the sheet: C23, C27
