File: H_bridge_PCB_Design/voltage_source.kicad_sch (KiCad schematic)
At the start: 27 parts, among them IC1 LM2671M-3.3_NOPB, IC2 L7812ABD2T-TR, J15 TSW-102-15-T-S, U6 LD1086DT50TR, U8 3544-2

Commit message: huge changes output measurement
Parts:
- removed C22: 100uF, SamacSys_Parts:EEE1AA101SP, symbol Device:C_Polarized_Small_US
- removed D13: S210, SamacSys_Parts:DIOM5336X265N, symbol SamacSys_Parts:S210
- removed IC1: LM2671M-3.3_NOPB, SOIC127P600X175-8N, symbol SamacSys_Parts:LM2671M-3.3_NOPB
- removed L1: IFDC3030EZER101M, SamacSys_Parts:IFDC3030EZER101M, symbol SamacSys_Parts:IFDC3030EZER101M
- added LED4: TLMG1100-GS15-1, Resistor_SMD:R_0805_2012Metric_Pad1.20x1.40mm_HandSolder, symbol SamacSys_Parts:TLMG1100-GS15
- added R11: 100, Resistor_SMD:R_0805_2012Metric_Pad1.20x1.40mm_HandSolder, symbol Device:R
- added U5: LT1963AxST-3.3, Package_TO_SOT_SMD:SOT-223-3_TabPin2, symbol Regulator_Linear:LT1963AxST-3.3
- C11: value 10 nF -> 1µF
Connections:
- net +3.3V: now also C11.1, U5.3 (OUT)
- net GND: now also C11.2, R11.1, U5.2 (GND)
- new net: LED4.1 (K), R11.2
- new net SatusLED: LED4.2 (A)
- new net VUSB(5V): U5.1 (IN)

Commit message: new pcb
Parts:
- removed U8: 3544-2, SamacSys_Parts:3544-2, symbol SamacSys_Parts:3544-2
- C11, C17, C21, C25, C26, C27: LCSC Part # (none) -> C28323; LCSC Part# C28323 -> (none)
- C23, C7, C8: LCSC Part # (none) -> C128464; LCSC Part# C128464 -> (none)
- IC2: LCSC Part # (none) -> C186698; LCSC Part# C186698 -> (none)
- LED1, LED2, LED3, LED4: LCSC Part # (none) -> C434436; LCSC Part# C434436 -> (none)
- R11, R27: LCSC Part # (none) -> C115423; LCSC Part# C115423 -> (none)
- R12, R29: LCSC Part # (none) -> C4129769; LCSC Part# C4129769 -> (none)
- R28: LCSC Part # (none) -> C95781; LCSC Part# C95781 -> (none)
- U5: LCSC Part # (none) -> C459918
- U6: LCSC Part # (none) -> C164853; LCSC Part# C164853 -> (none)
Connections:
- net +24V: now also TP1.1
